File: 555_I_delay.kicad_sch (KiCad schematic)
At the start: 18 parts, among them J1 I_In, J2 I_out, J3 GND_Conn, Q1 FQD11P06TM, U1 NE555P

Commit message: added BOM
Parts:
- D1: value TVS -> SZ1SMB15AT3G
- D2: value BZV55B15 -> SZ1SMB15AT3G
- J1: footprint Connector_PinHeader_1.00mm:PinHeader_1x01_P1.00mm_Vertical -> Connector_Pin:12_AWG_TH_Alex
- R4: value 100k (pulldown) -> 100k
- U1: value NE555P -> TLC555CP
Changed lines of the file:
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@@
 			)
 		)
-		(property "Description" "capacitor, small US symbol"
+		(property "Description" "Smoothing capacitor"
 			(at 123.19 77.47 0)
 			(hide yes)
@@
 			)
 		)
-		(property "Description" "capacitor, small US symbol"
+		(property "Description" "Smoothing Capacitor"
 			(at 130.81 64.77 0)
 			(hide yes)
@@
 			)
 		)
-		(property "Description" "capacitor, small US symbol"
+		(property "Description" "Pulls Trig to ground momenterily"
 			(at 110.49 110.49 0)
 			(hide yes)
@@
 			)
 		)
-		(property "Value" "TVS"
+		(property "Value" "SZ1SMB15AT3G"
 			(at 185.42 113.3474 90)
+			(hide yes)
 			(show_name no)
 			(do_not_autoplace no)
@@
 			)
 		)
-		(property "Datasheet" "https://www.vishay.com/docs/88751/ss32.pdf"
+		(property "Datasheet" ""
 			(at 182.88 111.76 0)
 			(hide yes)
@@
 			)
 		)
-		(property "Description" "30V 3A Schottky Diode, SMA"
+		(property "Description" "Gate/Drain TVS protection"
 			(at 182.88 111.76 0)
 			(hide yes)
@@
 			)
 		)
-		(property "Footprint" "Connector_PinHeader_1.00mm:PinHeader_1x01_P1.00mm_Vertical"
+		(property "Footprint" "Connector_Pin:12_AWG_TH_Alex"
 			(at 71.12 78.74 0)
 			(hide yes)
@@
 			)
 		)
-		(property "Description" "Generic connector, single row, 01x01, script generated"
+		(property "Description" "Wire Mounting hole"
 			(at 71.12 78.74 0)
 			(hide yes)
@@
 			)
 		)
-		(property "Description" "Resistor, small US symbol"
+		(property "Description" "Resistor for RC timing circuit"
 			(at 97.79 77.47 0)
 			(hide yes)
@@
 			)
 		)
-		(property "Description" "Resistor, small US symbol"
+		(property "Description" "Raises trig up after initial start"
 			(at 110.49 69.85 0)
 			(hide yes)
@@
 			)
 		)
-		(property "Value" "BZV55B15"
+		(property "Value" "SZ1SMB15AT3G"
 			(at 135.89 52.07 0)
+			(hide yes)
 			(show_name no)
 			(do_not_autoplace no)
@@
 			)
 		)
-		(property "Datasheet" "https://assets.nexperia.com/documents/data-sheet/BZV55_SER.pdf"
+		(property "Datasheet" ""
 			(at 135.89 55.88 0)
 			(hide yes)
@@
 			)
 		)
-		(property "Description" "15V, 500mW, 2%, Zener diode, MiniMELF"
+		(property "Description" "Supply voltage TVS"
 			(at 135.89 55.88 0)
 			(hide yes)
@@
 			)
 		)
-		(property "Description" "capacitor, small US symbol"
+		(property "Description" "Electrolytic capcitor for RC timing circuit"
 			(at 97.79 110.49 0)
 			(hide yes)
@@
 			)
 		)
-		(property "Description" "Generic connector, single row, 01x01, script generated"
+		(property "Description" "Chassis and circuit ground"
 			(at 130.81 113.03 0)
 			(hide yes)
@@
 			)
 		)
-		(property "Value" "NE555P"
+		(property "Value" "TLC555CP"
 			(at 138.43 90.0998 0)
+			(hide yes)
 			(show_name no)
 			(do_not_autoplace no)
@@
 			)
 		)
-		(property "Datasheet" "http://www.ti.com/lit/ds/symlink/ne555.pdf"
+		(property "Datasheet" ""
 			(at 125.73 120.65 0)
 			(hide yes)
@@
 			)
 		)
-		(property "Description" "Precision Timers, 555 compatible, PDIP-8"
+		(property "Description" "CMOS 555 compatible, PDIP-8"
 			(at 125.73 115.57 0)
 			(hide yes)
@@
 			)
 		)
-		(property "Value" "100k (pulldown)"
+		(property "Value" "100k"
 			(at 171.45 105.4099 0)
 			(show_name no)
@@
 			)
 		)
-		(property "Description" "Resistor, small US symbol"
+		(property "Description" "MOSFET pull-down resistor"
 			(at 168.91 104.14 0)
 			(hide yes)
@@
 		(property "Value" "Fuse_Small"
 			(at 78.74 66.0399 90)
+			(hide yes)
 			(show_name no)
 			(do_not_autoplace no)
@@
 			)
 		)
-		(property "Description" "Fuse, small symbol"
+		(property "Description" "Fuse, 10A"
 			(at 77.47 64.77 0)
 			(hide yes)
@@
 			)
 		)
-		(property "Description" "Resistor, small US symbol"
+		(property "Description" "Resistor to minimize line ringing"
 			(at 151.13 93.98 0)
 			(hide yes)
